File: ez-uart-adapter.kicad_pcb (KiCad board)
At the start: 2 copper layers, 45 x 15 mm, 23 parts, among them J1 USB_C_Receptacle_USB2.0_16P, J2 Conn_01x04_Pin, Q1 2N7002, Q2 2N7002, Q3 AO3401A, SW1 MK-11C04-G013, U1 USBLC6-2SC6, U2 AP2112K-3.3, U3 CH340C

Commit message: Fix orientation of LEDs
🤦
Parts:
- moved D2 0.52 mm to (166.7, 98.6), turned to 180 degrees
- turned D1 to 0 degrees
Connections:
- D1 pad 1: Net-(D1-K) -> GND
- D1 pad 2: GND -> Net-(D1-A)
- D2 pad 1: Net-(D2-K) -> GND
- D2 pad 2: GND -> Net-(D2-A)
- R1 pad 2: Net-(D1-K) -> Net-(D1-A)
- R8 pad 2: Net-(D2-K) -> Net-(D2-A)
Routing:
- net Net-(D2-K): track 2.56 -> 0.00 mm
- net Net-(D2-A): track 0.00 -> 2.56 mm
- net Net-(D1-K): track 2.00 -> 0.00 mm
- net Net-(D1-A): track 0.00 -> 2.00 mm
- net GND: track 19.3 -> 18.5 mm
Changed lines of the file:
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@@
 	(footprint "LED_SMD:LED_0603_1608Metric_Pad1.05x0.95mm_HandSolder"
 		(layer "F.Cu")
-		(at 128.6 98.7 180)
+		(at 128.6 98.7)
 		(descr "LED SMD 0603 (1608 Metric), square (rectangular) end terminal, IPC-7351 nominal, (Body size source: http://www.tortai-tech.com/upload/download/2011102023233369053.pdf)")
 		(tags "LED handsolder")
 		(property "Reference" "D1"
-			(at 0 -1.43 180)
+			(at 0 -1.43 0)
 			(layer "F.SilkS")
 			(hide yes)
@@
 		)
 		(property "Value" "red"
-			(at 0 -1 180)
+			(at 0 -1 0)
 			(layer "F.Fab")
 			(effects
@@
 		)
 		(property "Datasheet" ""
-			(at 0 0 180)
+			(at 0 0 0)
 			(layer "F.Fab")
 			(hide yes)
@@
 		)
 		(property "Description" "Light emitting diode"
-			(at 0 0 180)
+			(at 0 0 0)
 			(layer "F.Fab")
 			(hide yes)
@@
 		)
 		(property "KiLib_Generator" "SMD_2terminal_chip_molded"
-			(at 0 0 180)
+			(at 0 0 0)
 			(layer "F.SilkS")
 			(hide yes)
@@
 		)
 		(property "Sim.Pins" "1=K 2=A"
-			(at 0 0 180)
+			(at 0 0 0)
 			(unlocked yes)
 			(layer "F.Fab")
@@
 		)
 		(property "Dielectric" ""
-			(at 0 0 180)
+			(at 0 0 0)
 			(unlocked yes)
 			(layer "F.Fab")
@@
 		)
 		(property "Voltage" ""
-			(at 0 0 180)
+			(at 0 0 0)
 			(unlocked yes)
 			(layer "F.Fab")
@@
 		)
 		(property "LCSC Part" "C2286"
-			(at 0 0 180)
+			(at 0 0 0)
 			(unlocked yes)
 			(layer "F.Fab")
@@
 		(duplicate_pad_numbers_are_jumpers no)
 		(fp_line
-			(start 0.8 -0.735)
-			(end -1.66 -0.735)
+			(start -1.66 -0.735)
+			(end -1.66 0.735)
 			(stroke
 				(width 0.12)
@@
 		)
 		(fp_line
-			(start -1.66 -0.735)
-			(end -1.66 0.735)
+			(start 0.8 -0.735)
+			(end -1.66 -0.735)
 			(stroke
 				(width 0.12)
@@
 		)
 		(fp_line
-			(start 0.8 0.4)
-			(end 0.8 -0.4)
+			(start -0.8 -0.1)
+			(end -0.8 0.4)
 			(stroke
 				(width 0.1)
@@
 		)
 		(fp_line
-			(start 0.8 -0.4)
-			(end -0.5 -0.4)
+			(start -0.8 0.4)
+			(end 0.8 0.4)
 			(stroke
 				(width 0.1)
@@
 		)
 		(fp_line
-			(start -0.8 0.4)
-			(end 0.8 0.4)
+			(start 0.8 -0.4)
+			(end -0.5 -0.4)
 			(stroke
 				(width 0.1)
@@
 		)
 		(fp_line
-			(start -0.8 -0.1)
-			(end -0.8 0.4)
+			(start 0.8 0.4)
+			(end 0.8 -0.4)
 			(stroke
 				(width 0.1)
@@
 		)
 		(fp_text user "${REFERENCE}"
-			(at 0 0 180)
+			(at 0 0 0)
 			(layer "F.Fab")
 			(effects
@@
 		)
 		(pad "1" smd roundrect
-			(at -0.875 0 180)
+			(at -0.875 0)
 			(size 1.05 0.95)
 			(layers "F.Cu" "F.Mask" "F.Paste")
 			(roundrect_rratio 0.25)
-			(net "Net-(D1-K)")
+			(net "GND")
 			(pinfunction "K_1")
 			(pintype "passive")
 		)
 		(pad "2" smd roundrect
-			(at 0.875 0 180)
+			(at 0.875 0)
 			(size 1.05 0.95)
 			(layers "F.Cu" "F.Mask" "F.Paste")
 			(roundrect_rratio 0.25)
-			(net "GND")
+			(net "Net-(D1-A)")
 			(pinfunction "A_2")
 			(pintype "passive")
@@
 			(layers "F.Cu" "F.Mask" "F.Paste")
 			(roundrect_rratio 0.25)
-			(net "Net-(D1-K)")
+			(net "Net-(D1-A)")
 			(pintype "passive")
 		)
@@
 			(layers "F.Cu" "F.Mask" "F.Paste")
 			(roundrect_rratio 0.25)
-			(net "Net-(D2-K)")
+			(net "Net-(D2-A)")
 			(pintype "passive")
 		)
@@
 	(footprint "LED_SMD:LED_0603_1608Metric_Pad1.05x0.95mm_HandSolder"
 		(layer "F.Cu")
-		(at 167.2 98.6)
+		(at 166.675 98.6 180)
 		(descr "LED SMD 0603 (1608 Metric), square (rectangular) end terminal, IPC-7351 nominal, (Body size source: http://www.tortai-tech.com/upload/download/2011102023233369053.pdf)")
 		(tags "LED handsolder")
@@
 		)
 		(property "Sim.Pins" "1=K 2=A"
-			(at 0 0 0)
+			(at 0 0 180)
 			(unlocked yes)
 			(layer "F.Fab")
@@
 		)
 		(property "Dielectric" ""
-			(at 0 0 0)
+			(at 0 0 180)
 			(unlocked yes)
 			(layer "F.Fab")
@@
 		)
 		(property "Voltage" ""
-			(at 0 0 0)
+			(at 0 0 180)
 			(unlocked yes)
 			(layer "F.Fab")
@@
 		)
 		(property "LCSC Part" "C12624"
-			(at 0 0 0)
+			(at 0 0 180)
 			(unlocked yes)
 			(layer "F.Fab")
@@
 		(duplicate_pad_numbers_are_jumpers no)
 		(fp_line
-			(start -1.66 -0.735)
-			(end -1.66 0.735)
+			(start 0.8 -0.735)
+			(end -1.66 -0.735)
 			(stroke
 				(width 0.12)
@@
 		)
 		(fp_line
-			(start 0.8 -0.735)
-			(end -1.66 -0.735)
+			(start -1.66 -0.735)
+			(end -1.66 0.735)
 			(stroke
 				(width 0.12)
@@
 		)
 		(fp_line
-			(start -0.8 -0.1)
-			(end -0.8 0.4)
+			(start 0.8 0.4)
+			(end 0.8 -0.4)
 			(stroke
 				(width 0.1)
@@
 		)
 		(fp_line
-			(start -0.8 0.4)
-			(end 0.8 0.4)
+			(start 0.8 -0.4)
+			(end -0.5 -0.4)
 			(stroke
 				(width 0.1)
@@
 		)
 		(fp_line
-			(start 0.8 -0.4)
-			(end -0.5 -0.4)
+			(start -0.8 0.4)
+			(end 0.8 0.4)
 			(stroke
 				(width 0.1)
@@
 		)
 		(fp_line
-			(start 0.8 0.4)
-			(end 0.8 -0.4)
+			(start -0.8 -0.1)
+			(end -0.8 0.4)
 			(stroke
 				(width 0.1)
@@
 		)
 		(pad "1" smd roundrect
-			(at -0.875 0)
+			(at -0.875 0 180)
 			(size 1.05 0.95)
 			(layers "F.Cu" "F.Mask" "F.Paste")
 			(roundrect_rratio 0.25)
-			(net "Net-(D2-K)")
+			(net "GND")
 			(pinfunction "K_1")
 			(pintype "passive")
 		)
 		(pad "2" smd roundrect
-			(at 0.875 0)
+			(at 0.875 0 180)
 			(size 1.05 0.95)
 			(layers "F.Cu" "F.Mask" "F.Paste")
 			(roundrect_rratio 0.25)
-			(net "GND")
+			(net "Net-(D2-A)")
 			(pinfunction "A_2")
 			(pintype "passive")
@@
 	)
 	(segment
-		(start 129.1875 98.7)
-		(end 131.1875 98.7)
-		(width 0.2)
-		(layer "F.Cu")
-		(net "Net-(D1-K)")
-	)
-	(segment
 		(start 168.075 98.6)
-		(end 169.1 98.6)
+		(end 168.3 98.6)
 		(width 0.2)
 		(layer "F.Cu")
@@
 	)
 	(via
-		(at 169.1 98.6)
+		(at 168.6 98.6)
 		(size 0.6)
 		(drill 0.3)
@@
 	)
 	(segment
-		(start 163.6 98.675)
-		(end 166.0375 98.675)
-		(width 0.2)
-		(layer "F.Cu")
-		(net "Net-(D2-K)")
-	)
-	(segment
-		(start 166.0375 98.675)
-		(end 166.1125 98.6)
-		(width 0.2)
-		(layer "F.Cu")
-		(net "Net-(D2-K)")
-	)
-	(segment
-		(start 166.0125 98.5)
-		(end 166 98.5)
-		(width 0.2)
-		(layer "F.Cu")
-		(net "Net-(D2-K)")
-	)
-	(segment
 		(start 146.910682 106.045)
 		(end 146.635 106.045)
@@
 		(net "Net-(U3-~{DTR})")
 	)
+	(segment
+		(start 129.1875 98.7)
+		(end 131.1875 98.7)
+		(width 0.2)
+		(layer "F.Cu")
+		(net "Net-(D1-A)")
+	)
+	(segment
+		(start 163.6 98.675)
+		(end 166.0375 98.675)
+		(width 0.2)
+		(layer "F.Cu")
+		(net "Net-(D2-A)")
+	)
+	(segment
+		(start 166.0375 98.675)
+		(end 166.1125 98.6)
+		(width 0.2)
+		(layer "F.Cu")
+		(net "Net-(D2-A)")
+	)
+	(segment
+		(start 166.0125 98.5)
+		(end 166 98.5)
+		(width 0.2)
+		(layer "F.Cu")
+		(net "Net-(D2-A)")
+	)
 	(zone

Commit message: Add ESD protection to UART
Parts:
- added R10: 470R, Resistor_SMD:R_0603_1608Metric_Pad0.98x0.95mm_HandSolder, F.Cu at (164.4, 108.9)
- added R9: 470R, Resistor_SMD:R_0603_1608Metric_Pad0.98x0.95mm_HandSolder, F.Cu at (164.4, 104.7)
- moved SW1 2.20 mm to (159.2, 110.1)
- moved D2 0.52 mm to (167.2, 98.6), turned to 0 degrees
- turned D1 to 180 degrees
Connections:
- D1 pad 1: GND -> Net-(D1-K)
- D1 pad 2: Net-(D1-A) -> GND
- D2 pad 1: GND -> Net-(D2-K)
- D2 pad 2: Net-(D2-A) -> GND
- J2 pad 2: RX -> Net-(J2-Pin_2)
- J2 pad 3: TX -> Net-(J2-Pin_3)
- R1 pad 2: Net-(D1-A) -> Net-(D1-K)
- R8 pad 2: Net-(D2-A) -> Net-(D2-K)
Routing:
- net RX: track 34.0 -> 28.6 mm
- net TX: track 36.6 -> 32.0 mm
- net Net-(J2-Pin_2): track 0.00 -> 3.22 mm
- net Net-(J2-Pin_3): track 0.00 -> 2.81 mm
- net Net-(D2-K): track 0.00 -> 2.56 mm
- net Net-(D2-A): track 2.56 -> 0.00 mm
- net Net-(D1-K): track 0.00 -> 2.00 mm
- net Net-(D1-A): track 2.00 -> 0.00 mm
- net Net-(Q3-G): track 11.5 -> 12.4 mm
- net GND: track 18.5 -> 19.3 mm
